Commit message: simulation-wcr_description: Model now able to move and has one functioning lidar-sensor

File: simulation-wcr_description/urdf/wheelchair-robot.urdf (robot description, URDF)
Before this commit: robot wheelchair-robot-fhws, 6 links, 5 joints
Links:
- added link lidar, mass 0.125; collision cylinder length=0.055 radius=0.0508; visual mesh filename=package://simulation-wcr_description/meshes/lds.dae scale=0.001 0.001 0.001
Joints:
- added joint lidar_joint: type fixed, parent wcr_base_link, child lidar, origin xyz=0.535 0.2875 0.187 rpy=0 0 0

File: simulation-wcr_description/urdf/wheelchair-robot.xacro (robot description, xacro)
@@ -16,4 +16,8 @@
     <child link="wcr_base_link" />
   </joint>
+  <gazebo reference="base_link">
+    <material>Gazebo/Yellow</material>
+    <gravity>true</gravity>
+  </gazebo>
   <link name="wcr_base_link">
     <visual>
@@ -40,4 +44,7 @@
     </inertial>
   </link>
+  <gazebo reference="wcr_base_link">
+    <material>Gazebo/Yellow</material>
+  </gazebo>
   <joint name="upper_left_wheel_joint" type="continuous">
     <origin xyz="0.455 0.2925 0.03" rpy="0 0 0" />
@@ -156,3 +163,132 @@
     </inertial>
   </link>
+  <gazebo reference="upper_left_mecanum_wheel">
+    <material>Gazebo/Grey</material>
+  </gazebo>
+  <gazebo reference="lower_left_mecanum_wheel">
+    <material>Gazebo/DarkGrey</material>
+  </gazebo>
+  <gazebo reference="upper_right_mecanum_wheel">
+    <material>Gazebo/DarkGrey</material>
+  </gazebo>
+  <gazebo reference="lower_right_mecanum_wheel">
+    <material>Gazebo/Grey</material>
+  </gazebo>
+  <joint name="lidar_joint" type="fixed">
+    <origin xyz="0.535 0.2875 0.155" rpy="0 0 0" />
+    <parent link="wcr_base_link"/>
+    <child link="lidar" />
+  </joint>
+  <link name="lidar">
+    <visual>
+      <origin xyz="0 0 0" rpy="0 0 0" />
+      <geometry>
+        <mesh filename="package://simulation-wcr_description/meshes/rplidar-a2m4-r1.stl" scale="0.001 0.001 0.001"/>
+      </geometry>
+      <material name="black" />
+    </visual>
+    <collision>
+      <origin xyz="0 0 0.0204" rpy="0 0 0"/>
+      <geometry>
+        <cylinder radius="0.045" length="0.05"/>
+      </geometry>
+    </collision>
+    <inertial>
+      <origin xyz="0 0 0" rpy="0 0 0"/>
+      <mass value="0.125"/>
+      <inertia
+        ixx="0.001" ixy="0.0000" ixz="0.00000"
+        iyy="0.001" iyz="0.000"
+        izz="0.001"/>
+    </inertial>
+  </link>
+  <gazebo reference="lidar">
+    <sensor type="ray" name="RPLiDAR_A2M8">
+      <pose>0 0 0.0308 0 0 0</pose>
+      <always_on>true</always_on>
+      <visualize>false</visualize>
+      <update_rate>1800</update_rate>
+      <ray>
+        <scan>
+          <horizontal>
+            <samples>400</samples>
+            <resolution>1</resolution>
+            <min_angle>0</min_angle>
+            <max_angle>6.280</max_angle>
+          </horizontal>
+        </scan>
+        <range>
+          <min>0.15</min>
+          <max>8.0</max>
+          <resolution>0.008</resolution>
+        </range>
+        <noise>
+          <type>gaussian</type>
+          <mean>0.0</mean>
+          <stddev>0.01</stddev>
+        </noise>
+      </ray>
+      <plugin name="RPLiDAR_A2M8_measurement" filename="libgazebo_ros_laser.so">
+        <topicName>/lidar_scan</topicName>
+        <frameName>RPLiDAR</frameName>
+      </plugin>
+    </sensor>
+  </gazebo>
+  <gazebo reference="lidar">
+    <material>Gazebo/Black</material>
+  </gazebo>
+  <!-- Linking Gazebo and ROS-->
+  <gazebo>
+    <plugin name="gazebo_ros_control" filename="libgazebo_ros_control.so">
+      <robotNamespace>/</robotNamespace>
+    </plugin>
+  </gazebo>
+  <!--Including planar movement in order to imitate omidirectional movement with mecanum wheels-->
+  <gazebo>
+    <plugin name="object_controller" filename="libgazebo_ros_planar_move.so">
+      <commandTopic>cmd_vel</commandTopic>
+      <odometryTopic>odom</odometryTopic>
+      <odometryFrame>odom</odometryFrame>
+      <odometryRate>20.0</odometryRate>
+      <robotBaseFrame>base_link</robotBaseFrame>
+    </plugin>
+  </gazebo>
+  <!-- This block connects joints to actuator (dc motors), which informs both
+  simulation and visualization of the robot. Only used for showing model right in RViZ.-->
+  <transmission name="left_front_wheel">
+    <type>transmission_interface/SimpleTransmission</type>
+    <actuator name="$left_front_dc_motor">
+      <mechanicalReduction>1</mechanicalReduction>
+    </actuator>
+    <joint name="upper_left_wheel_joint">
+      <hardwareInterface>hardware_interface/PositionJointInterface</hardwareInterface>
+    </joint>
+  </transmission>
+  <transmission name="left_back_wheel">
+    <type>transmission_interface/SimpleTransmission</type>
+    <actuator name="$left_back_dc_motor">
+      <mechanicalReduction>1</mechanicalReduction>
+    </actuator>
+    <joint name="lower_left_wheel_joint">
+      <hardwareInterface>hardware_interface/PositionJointInterface</hardwareInterface>
+    </joint>
+  </transmission>
+  <transmission name="right_front_wheel">
+    <type>transmission_interface/SimpleTransmission</type>
+    <actuator name="$right_front_dc_motor">
+      <mechanicalReduction>1</mechanicalReduction>
+    </actuator>
+    <joint name="upper_right_wheel_joint">
+      <hardwareInterface>hardware_interface/PositionJointInterface</hardwareInterface>
+    </joint>
+  </transmission>
+  <transmission name="right_back_wheel">
+    <type>transmission_interface/SimpleTransmission</type>
+    <actuator name="$right_back_dc_motor">
+      <mechanicalReduction>1</mechanicalReduction>
+    </actuator>
+    <joint name="lower_right_wheel_joint">
+      <hardwareInterface>hardware_interface/PositionJointInterface</hardwareInterface>
+    </joint>
+  </transmission>
 </robot>

Commit message: simulation-wcr_description: Lidar Sensor now works as intended

File: simulation-wcr_description/urdf/wheelchair-robot.urdf (robot description, URDF)
Before this commit: robot wheelchair-robot-fhws, 7 links, 6 joints
Links:
- link lidar: geometry collision cylinder length=0.05 radius=0.045; visual mesh filename=package://simulation-wcr_description/meshes/rplidar-a2m4-r1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 scale=0.001 0.001 0.001
Joints:
- joint lidar_joint: origin xyz=0.535 0.2875 0.187 rpy=0 0 0 -> xyz=0.535 0.2875 0.1838 rpy=0 0 0

File: simulation-wcr_description/urdf/wheelchair-robot.xacro (robot description, xacro)
@@ -176,5 +176,5 @@
   </gazebo>
   <joint name="lidar_joint" type="fixed">
-    <origin xyz="0.535 0.2875 0.155" rpy="0 0 0" />
+    <origin xyz="0.535 0.2875 0.1838" rpy="0 0 0" />
     <parent link="wcr_base_link"/>
     <child link="lidar" />
@@ -182,5 +182,5 @@
   <link name="lidar">
     <visual>
-      <origin xyz="0 0 0" rpy="0 0 0" />
+      <origin xyz="0 0 -0.0308" rpy="0 0 0" />
       <geometry>
         <mesh filename="package://simulation-wcr_description/meshes/rplidar-a2m4-r1.stl" scale="0.001 0.001 0.001"/>
@@ -189,5 +189,5 @@
     </visual>
     <collision>
-      <origin xyz="0 0 0.0204" rpy="0 0 0"/>
+      <origin xyz="0 0 -0.0104" rpy="0 0 0"/>
       <geometry>
         <cylinder radius="0.045" length="0.05"/>
@@ -205,8 +205,8 @@
   <gazebo reference="lidar">
     <sensor type="ray" name="RPLiDAR_A2M8">
-      <pose>0 0 0.0308 0 0 0</pose>
+      <pose>0 0 0 0 0 0</pose>
       <always_on>true</always_on>
       <visualize>false</visualize>
-      <update_rate>1800</update_rate>
+      <update_rate>100</update_rate>
       <ray>
         <scan>
@@ -214,6 +214,6 @@
             <samples>400</samples>
             <resolution>1</resolution>
-            <min_angle>0</min_angle>
-            <max_angle>6.280</max_angle>
+            <min_angle>0.0</min_angle>
+            <max_angle>6.28319</max_angle>
           </horizontal>
         </scan>
@@ -221,10 +221,10 @@
           <min>0.15</min>
           <max>8.0</max>
-          <resolution>0.008</resolution>
+          <resolution>0.08</resolution>
         </range>
         <noise>
           <type>gaussian</type>
           <mean>0.0</mean>
-          <stddev>0.01</stddev>
+          <stddev>0.015</stddev> <!--stddev needs to be checked again-->
         </noise>
       </ray>
