Commit message: simulation-wcr_description: deleted base_foot link because it is not needed, added a second simulation with two lidars slam_algorithms: added launch files for algorithms with merged laser data (merged laser data does not work properly in this version)

File: simulation-wcr_description/urdf/wheelchair-robot_two_lidar.xacro (robot description, xacro)
@@ -163,10 +163,38 @@
     <material>Gazebo/Grey</material>
   </gazebo>
-  <joint name="lidar_joint" type="fixed">
+  <joint name="lidar_joint_front" type="fixed">
     <origin xyz="0.535 0.2875 0.1838" rpy="0 0 0" />
     <parent link="base_link"/>
-    <child link="lidar" />
-  </joint>
-  <link name="lidar">
+    <child link="lidar_front" />
+  </joint>
+  <link name="lidar_front">
+    <visual>
+      <origin xyz="0 0 -0.0308" rpy="0 0 0" />
+      <geometry>
+        <mesh filename="package://simulation-wcr_description/meshes/rplidar-a2m4-r1.stl" scale="0.001 0.001 0.001"/>
+      </geometry>
+      <material name="black" />
+    </visual>
+    <collision>
+      <origin xyz="0 0 -0.0104" rpy="0 0 0"/>
+      <geometry>
+        <cylinder radius="0.045" length="0.05"/>
+      </geometry>
+    </collision>
+    <inertial>
+      <origin xyz="0 0 0" rpy="0 0 0"/>
+      <mass value="0.125"/>
+      <inertia
+        ixx="0.001" ixy="0.0000" ixz="0.00000"
+        iyy="0.001" iyz="0.000"
+        izz="0.001"/>
+    </inertial>
+  </link>
+  <joint name="lidar_joint_back" type="fixed">
+    <origin xyz="-0.535 -0.2875 0.2138" rpy="0 0 3.141593" />
+    <parent link="base_link"/>
+    <child link="lidar_back" />
+  </joint>
+  <link name="lidar_back">
     <visual>
       <origin xyz="0 0 -0.0308" rpy="0 0 0" />
@@ -209,6 +237,6 @@
   </gazebo>
 <!--Below is the code/plug-in for a LiDAR sensor-->
-  <gazebo reference="lidar">
-    <sensor type="ray" name="RPLiDAR_A2M8">
+  <gazebo reference="lidar_front">
+    <sensor type="ray" name="RPLiDAR_A2M8_front">
       <pose>0 0 0 0 0 0</pose>
       <always_on>true</always_on>
@@ -235,11 +263,46 @@
         </noise>
       </ray>
-      <plugin name="RPLiDAR_A2M8_measurement" filename="libgazebo_ros_laser.so">
-        <topicName>/lidar_scan</topicName>
-        <frameName>lidar</frameName>
+      <plugin name="RPLiDAR_A2M8_measurement_front" filename="libgazebo_ros_laser.so">
+        <topicName>/lidar_scan_front</topicName>
+        <frameName>lidar_front</frameName>
       </plugin>
     </sensor>
   </gazebo>
-  <gazebo reference="lidar">
+  <gazebo reference="lidar_front">
+    <material>Gazebo/Black</material>
+  </gazebo>
+  <gazebo reference="lidar_back">
+    <sensor type="ray" name="RPLiDAR_A2M8_back">
+      <pose>0 0 0 0 0 0</pose>
+      <always_on>true</always_on>
+      <visualize>true</visualize>
+      <update_rate>10</update_rate>
+      <ray>
+        <scan>
+          <horizontal>
+            <samples>400</samples>
+            <resolution>1</resolution>
+            <min_angle>-1.570796</min_angle> <!--using a field of 270 degrees on one corner (-177° to 90° in Simulation because of the CAD model with LiDAR space in the back)-->
+            <max_angle>3.141593</max_angle>
+          </horizontal>
+        </scan>
+        <range>
+          <min>0.15</min>
+          <max>8.0</max>
+          <resolution>0.08</resolution> <!--datasheet only contains resolution no accuracy-->
+        </range>
+        <noise>
+          <type>gaussian</type>
+          <mean>0.0</mean>
+          <stddev>0.02667</stddev> <!--stddev for A2M8-R2 is 0.08/3 (using resolution)-->
+        </noise>
+      </ray>
+      <plugin name="RPLiDAR_A2M8_measurement_back" filename="libgazebo_ros_laser.so">
+        <topicName>/lidar_scan_back</topicName>
+        <frameName>lidar_back</frameName>
+      </plugin>
+    </sensor>
+  </gazebo>
+  <gazebo reference="lidar_back">
     <material>Gazebo/Black</material>
   </gazebo>

Commit message: slam_algorithms: merging of both lidar values into one is now workiing. Mapping ist not possible at this moment due to an other occuring error

File: simulation-wcr_description/urdf/wheelchair-robot_two_lidar.xacro (robot description, xacro)
@@ -12,5 +12,5 @@
   </link>
   <joint name="base_joint" type="fixed">
-    <origin xyz="0 0 0.0" rpy="0 0 0" />
+    <origin xyz="0 0 0" rpy="0 0 0" />
     <parent link="base_foot"/>
     <child link="base_link" />
@@ -231,4 +231,13 @@
     </inertial>
   </link>
+<!--
+  <joint name="lidar_merge_joint" type="fixed">
+    <origin xyz="0 0 0.1988" rpy="0 0 0" />
+    <parent link="base_link"/>
+    <child link="lidar_merge_link" />
+  </joint>
+  <link name="lidar_merge_link">
+    <origin xyz="0 0 0" rpy="0 0 0" />
+  </link> -->
   <!-- Linking Gazebo and ROS-->
   <gazebo>
