Commit message: changed the links and joints in the simulation-wcr_description package (for the simulation), added a folder with launch and initialization files for karto, gmapping, and google cartographer slam algorithms

File: simulation-wcr_description/urdf/wheelchair-robot.xacro (robot description, xacro)
@@ -257,5 +257,13 @@
   </gazebo>
   <!--Below is the code/plug-in for a IMU (which at first won't be used)-->
-  <gazebo reference="wcr_base_link">
+  <joint name="imu_joint" type="fixed">
+    <origin xyz="0 0 0.227" rpy="0 0 0" />
+    <parent link="base_link"/>
+    <child link="imu_link" />
+  </joint>
+  <link name="imu_link">
+    <origin xyz="0 0 0" rpy="0 0 0" />
+  </link>
+  <gazebo reference="imu_link">
     <gravity>true</gravity>
     <sensor name="imu_sensor_wcr" type="imu">

Commit message: simulation-wcr_description: readded base_foot because of possible warning of inertia of base link.

File: simulation-wcr_description/urdf/wheelchair-robot.xacro (robot description, xacro)
@@ -8,4 +8,16 @@
   <material name="dark_grey"><color rgba="0.2 0.2 0.2 1.0" /></material>
   <material name="light_grey"><color rgba="0.4 0.4 0.4 1.0" /></material>
+  <link name="base_foot">
+    <origin xyz="0 0 0.07" rpy="0 0 0" />
+  </link>
+  <joint name="base_joint" type="fixed">
+    <origin xyz="0 0 0" rpy="0 0 0" />
+    <parent link="base_foot"/>
+    <child link="base_link" />
+  </joint>
+  <gazebo reference="base_foot">
+    <material>Gazebo/Yellow</material>
+    <gravity>true</gravity>
+  </gazebo>
   <link name="base_link">
     <visual>
@@ -204,5 +216,5 @@
       <odometryFrame>odom</odometryFrame>
       <odometryRate>100.0</odometryRate> <!-- Needs to be evaluated with the real one-->
-      <robotBaseFrame>base_link</robotBaseFrame>
+      <robotBaseFrame>base_foot</robotBaseFrame>
       <cmdTimeout>10.0</cmdTimeout>
     </plugin>

File: simulation-wcr_description/urdf/wheelchair-robot_two_lidar.xacro (robot description, xacro)
@@ -8,4 +8,16 @@
   <material name="dark_grey"><color rgba="0.2 0.2 0.2 1.0" /></material>
   <material name="light_grey"><color rgba="0.4 0.4 0.4 1.0" /></material>
+  <link name="base_foot">
+    <origin xyz="0 0 0.07" rpy="0 0 0" />
+  </link>
+  <joint name="base_joint" type="fixed">
+    <origin xyz="0 0 0.0" rpy="0 0 0" />
+    <parent link="base_foot"/>
+    <child link="base_link" />
+  </joint>
+  <gazebo reference="base_foot">
+    <material>Gazebo/Yellow</material>
+    <gravity>true</gravity>
+  </gazebo>
   <link name="base_link">
     <visual>
@@ -232,5 +244,5 @@
       <odometryFrame>odom</odometryFrame>
       <odometryRate>100.0</odometryRate> <!-- Needs to be evaluated with the real one-->
-      <robotBaseFrame>base_link</robotBaseFrame>
+      <robotBaseFrame>base_foot</robotBaseFrame>
       <cmdTimeout>10.0</cmdTimeout>
     </plugin>

Commit message: simulation_wcr_description/slam_algorithms: all errors have been removed and the simulation with two lidar sensors as well as the slam algorithms using two lidar sensorsr are now working

File: simulation-wcr_description/urdf/wheelchair-robot.xacro (robot description, xacro)
@@ -230,5 +230,5 @@
         <scan>
           <horizontal>
-            <samples>300</samples>
+            <samples>296</samples>
             <resolution>1</resolution>
             <min_angle>-1.570796</min_angle> <!--using a field of 270 degrees on one corner (-177° to 90° in Simulation because of the CAD model with LiDAR space in the back)-->

File: simulation-wcr_description/urdf/wheelchair-robot_two_lidar.xacro (robot description, xacro)
@@ -231,5 +231,4 @@
     </inertial>
   </link>
-<!--
   <joint name="lidar_merge_joint" type="fixed">
     <origin xyz="0 0 0.1988" rpy="0 0 0" />
@@ -239,5 +238,5 @@
   <link name="lidar_merge_link">
     <origin xyz="0 0 0" rpy="0 0 0" />
-  </link> -->
+  </link>
   <!-- Linking Gazebo and ROS-->
   <gazebo>
@@ -267,5 +266,5 @@
         <scan>
           <horizontal>
-            <samples>300</samples>
+            <samples>296</samples>
             <resolution>1</resolution>
             <min_angle>-1.570796</min_angle> <!--using a field of 270 degrees on one corner (-177° to 90° in Simulation because of the CAD model with LiDAR space in the back)-->
