Commit message: simulation-wcr_description: Changed the two_lidar simulation of the wheelchair robot so that the lidar-tfs are orientied like on the real robot

File: simulation-wcr_description/urdf_xacro/wheelchair-robot_two_lidar.xacro (robot description, xacro)
@@ -176,5 +176,5 @@
   </gazebo>
   <joint name="lidar_joint_front" type="fixed">
-    <origin xyz="0.535 0.2875 0.1838" rpy="0 0 0" />
+    <origin xyz="0.535 0.2875 0.1838" rpy="3.14159 3.14159 0.785398" />
     <parent link="base_link"/>
     <child link="lidar_front" />
@@ -204,5 +204,5 @@
   </link>
   <joint name="lidar_joint_back" type="fixed">
-    <origin xyz="-0.535 -0.2875 0.2138" rpy="0 0 3.141593" />
+    <origin xyz="-0.535 -0.2875 0.2138" rpy="0 0 0.785399" />
     <parent link="base_link"/>
     <child link="lidar_back" />
@@ -261,18 +261,18 @@
       <pose>0 0 0 0 0 0</pose>
       <always_on>true</always_on>
-      <visualize>true</visualize>
+      <visualize>false</visualize>
       <update_rate>10</update_rate>
       <ray>
         <scan>
           <horizontal>
-            <samples>296</samples>
+            <samples>400</samples>
             <resolution>1</resolution>
-            <min_angle>-1.570796</min_angle> <!--using a field of 270 degrees on one corner (-177° to 90° in Simulation because of the CAD model with LiDAR space in the back)-->
-            <max_angle>3.089233</max_angle>
+            <min_angle>-3.1415</min_angle> <!--using a field of 270 degrees on one corner (-177° to 90° in Simulation because of the CAD model with LiDAR space in the back)-->
+            <max_angle>3.1415</max_angle>
           </horizontal>
         </scan>
         <range>
           <min>0.15</min>
-          <max>8.0</max>
+          <max>12.0</max>
           <resolution>0.08</resolution> <!--datasheet only contains resolution no accuracy-->
         </range>
@@ -296,13 +296,13 @@
       <pose>0 0 0 0 0 0</pose>
       <always_on>true</always_on>
-      <visualize>true</visualize>
+      <visualize>false</visualize>
       <update_rate>10</update_rate>
       <ray>
         <scan>
           <horizontal>
-            <samples>300</samples>
+            <samples>400</samples>
             <resolution>1</resolution>
-            <min_angle>-1.570796</min_angle> <!--using a field of 270 degrees on one corner (-177° to 90° in Simulation because of the CAD model with LiDAR space in the back)-->
-            <max_angle>3.141593</max_angle>
+            <min_angle>-3.1415</min_angle>
+            <max_angle>3.1415</max_angle>
           </horizontal>
         </scan>
